File: pcb/memory.kicad_sch (KiCad schematic)
At the start: 4 parts, among them U3 W25Q32JVSSIQ_C179173

Commit message: asigning the footprints
Parts:
- C3: renamed from C1; footprint Package_SON:Winbond_USON-8-1EP_3x2mm_P0.5mm_EP0.2x1.6mm -> Capacitor_SMD:C_0603_1608Metric; LCSC Part (none) -> C1591
- R8: renamed from R3; footprint (none) -> Resistor_SMD:R_0603_1608Metric
- R9: renamed from R2; footprint Package_SON:Winbond_USON-8-1EP_3x2mm_P0.5mm_EP0.2x1.6mm -> Resistor_SMD:R_0603_1608Metric
Changed lines of the file:
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@@
 		(dnp no)
 		(fields_autoplaced yes)
-		(property "Reference" "#PWR07"
+		(property "Reference" "#PWR016"
 			(at 125.73 121.92 0)
 			(hide yes)
@@
 			(project "pcb"
 				(path "/7be3b359-5856-4193-92cd-ba6762ca843a/b50e6f0a-6f96-4eef-b3c8-9a37cc161327"
-					(reference "#PWR07")
+					(reference "#PWR016")
 					(unit 1)
 				)
@@
 		(dnp no)
 		(fields_autoplaced yes)
-		(property "Reference" "R3"
+		(property "Reference" "R8"
 			(at 127 101.5999 0)
 			(show_name no)
@@
 			)
 		)
-		(property "Footprint" ""
+		(property "Footprint" "Resistor_SMD:R_0603_1608Metric"
 			(at 122.682 102.87 90)
 			(hide yes)
@@
 		)
 		(property "Description" "Resistor"
+			(at 124.46 102.87 0)
+			(hide yes)
+			(show_name no)
+			(do_not_autoplace no)
+			(effects
+				(font
+					(size 1.27 1.27)
+				)
+			)
+		)
+		(property "KLC_S3.3" ""
+			(at 124.46 102.87 0)
+			(hide yes)
+			(show_name no)
+			(do_not_autoplace no)
+			(effects
+				(font
+					(size 1.27 1.27)
+				)
+			)
+		)
+		(property "KLC_S4.1" ""
+			(at 124.46 102.87 0)
+			(hide yes)
+			(show_name no)
+			(do_not_autoplace no)
+			(effects
+				(font
+					(size 1.27 1.27)
+				)
+			)
+		)
+		(property "KLC_S4.2_DVDD" ""
+			(at 124.46 102.87 0)
+			(hide yes)
+			(show_name no)
+			(do_not_autoplace no)
+			(effects
+				(font
+					(size 1.27 1.27)
+				)
+			)
+		)
+		(property "KLC_S4.2_VREG_VOUT" ""
 			(at 124.46 102.87 0)
 			(hide yes)
@@
 			(project "pcb"
 				(path "/7be3b359-5856-4193-92cd-ba6762ca843a/b50e6f0a-6f96-4eef-b3c8-9a37cc161327"
-					(reference "R3")
+					(reference "R8")
 					(unit 1)
 				)
@@
 		(dnp no)
 		(fields_autoplaced yes)
-		(property "Reference" "#PWR04"
+		(property "Reference" "#PWR017"
 			(at 179.07 100.33 0)
 			(hide yes)
@@
 			(project "pcb"
 				(path "/7be3b359-5856-4193-92cd-ba6762ca843a/b50e6f0a-6f96-4eef-b3c8-9a37cc161327"
-					(reference "#PWR04")
+					(reference "#PWR017")
 					(unit 1)
 				)
@@
 		(dnp no)
 		(fields_autoplaced yes)
-		(property "Reference" "#PWR08"
+		(property "Reference" "#PWR015"
 			(at 124.46 102.87 0)
 			(hide yes)
@@
 			(project "pcb"
 				(path "/7be3b359-5856-4193-92cd-ba6762ca843a/b50e6f0a-6f96-4eef-b3c8-9a37cc161327"
-					(reference "#PWR08")
+					(reference "#PWR015")
 					(unit 1)
 				)
@@
 		(dnp no)
 		(fields_autoplaced yes)
-		(property "Reference" "#PWR05"
+		(property "Reference" "#PWR018"
 			(at 193.04 102.87 0)
 			(hide yes)
@@
 			(project "pcb"
 				(path "/7be3b359-5856-4193-92cd-ba6762ca843a/b50e6f0a-6f96-4eef-b3c8-9a37cc161327"
-					(reference "#PWR05")
+					(reference "#PWR018")
 					(unit 1)
 				)
@@
 			)
 		)
+		(property "KLC_S3.3" ""
+			(at 152.4 111.76 0)
+			(hide yes)
+			(show_name no)
+			(do_not_autoplace no)
+			(effects
+				(font
+					(size 1.27 1.27)
+				)
+			)
+		)
+		(property "KLC_S4.1" ""
+			(at 152.4 111.76 0)
+			(hide yes)
+			(show_name no)
+			(do_not_autoplace no)
+			(effects
+				(font
+					(size 1.27 1.27)
+				)
+			)
+		)
+		(property "KLC_S4.2_DVDD" ""
+			(at 152.4 111.76 0)
+			(hide yes)
+			(show_name no)
+			(do_not_autoplace no)
+			(effects
+				(font
+					(size 1.27 1.27)
+				)
+			)
+		)
+		(property "KLC_S4.2_VREG_VOUT" ""
+			(at 152.4 111.76 0)
+			(hide yes)
+			(show_name no)
+			(do_not_autoplace no)
+			(effects
+				(font
+					(size 1.27 1.27)
+				)
+			)
+		)
 		(pin "1"
 		)
@@
 		(dnp no)
 		(fields_autoplaced yes)
-		(property "Reference" "R2"
+		(property "Reference" "R9"
 			(at 194.31 106.68 90)
 			(show_name no)
@@
 			)
 		)
-		(property "Footprint" "Package_SON:Winbond_USON-8-1EP_3x2mm_P0.5mm_EP0.2x1.6mm"
+		(property "Footprint" "Resistor_SMD:R_0603_1608Metric"
 			(at 194.31 114.808 90)
 			(hide yes)
@@
 		(property "Description" "Resistor"
 			(at 194.31 113.03 0)
+			(hide yes)
+			(show_name no)
+			(do_not_autoplace no)
+			(effects
+				(font
+					(size 1.27 1.27)
+				)
+			)
+		)
+		(property "KLC_S3.3" ""
+			(at 194.31 113.03 90)
+			(hide yes)
+			(show_name no)
+			(do_not_autoplace no)
+			(effects
+				(font
+					(size 1.27 1.27)
+				)
+			)
+		)
+		(property "KLC_S4.1" ""
+			(at 194.31 113.03 90)
+			(hide yes)
+			(show_name no)
+			(do_not_autoplace no)
+			(effects
+				(font
+					(size 1.27 1.27)
+				)
+			)
+		)
+		(property "KLC_S4.2_DVDD" ""
+			(at 194.31 113.03 90)
+			(hide yes)
+			(show_name no)
+			(do_not_autoplace no)
+			(effects
+				(font
+					(size 1.27 1.27)
+				)
+			)
+		)
+		(property "KLC_S4.2_VREG_VOUT" ""
+			(at 194.31 113.03 90)
 			(hide yes)
 			(show_name no)
@@
 			(project "pcb"
 				(path "/7be3b359-5856-4193-92cd-ba6762ca843a/b50e6f0a-6f96-4eef-b3c8-9a37cc161327"
-					(reference "R2")
+					(reference "R9")
 					(unit 1)
 				)
@@
 		(in_pos_files yes)
 		(dnp no)
-		(property "Reference" "C1"
+		(property "Reference" "C3"
 			(at 182.88 96.266 90)
 			(show_name no)
@@
 			)
 		)
-		(property "Footprint" "Package_SON:Winbond_USON-8-1EP_3x2mm_P0.5mm_EP0.2x1.6mm"
+		(property "Footprint" "Capacitor_SMD:C_0603_1608Metric"
 			(at 186.69 101.9048 0)
 			(hide yes)
@@
 		(property "Description" "Unpolarized capacitor"
 			(at 182.88 102.87 0)
+			(hide yes)
+			(show_name no)
+			(do_not_autoplace no)
+			(effects
+				(font
+					(size 1.27 1.27)
+				)
+			)
+		)
+		(property "KLC_S3.3" ""
+			(at 182.88 102.87 90)
+			(hide yes)
+			(show_name no)
+			(do_not_autoplace no)
+			(effects
+				(font
+					(size 1.27 1.27)
+				)
+			)
+		)
+		(property "KLC_S4.1" ""
+			(at 182.88 102.87 90)
+			(hide yes)
+			(show_name no)
+			(do_not_autoplace no)
+			(effects
+				(font
+					(size 1.27 1.27)
+				)
+			)
+		)
+		(property "KLC_S4.2_DVDD" ""
+			(at 182.88 102.87 90)
+			(hide yes)
+			(show_name no)
+			(do_not_autoplace no)
+			(effects
+				(font
+					(size 1.27 1.27)
+				)
+			)
+		)
+		(property "KLC_S4.2_VREG_VOUT" ""
+			(at 182.88 102.87 90)
+			(hide yes)
+			(show_name no)
+			(do_not_autoplace no)
+			(effects
+				(font
+					(size 1.27 1.27)
+				)
+			)
+		)
+		(property "LCSC Part" "C1591"
+			(at 182.88 102.87 90)
 			(hide yes)
 			(show_name no)
@@
 			(project "pcb"
 				(path "/7be3b359-5856-4193-92cd-ba6762ca843a/b50e6f0a-6f96-4eef-b3c8-9a37cc161327"
-					(reference "C1")
+					(reference "C3")
 					(unit 1)
 				)

Commit message: asigning the part numbers
Parts:
- R8: LCSC Part (none) -> C98220
- R9: LCSC Part (none) -> C23345
Changed lines of the file:
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@@
+			)
+		)
+		(property "LCSC Part" "C98220"
+			(at 124.46 102.87 0)
+			(hide yes)
+			(show_name no)
+			(do_not_autoplace no)
+			(effects
+				(font
+					(size 1.27 1.27)
+				)
 			)
 		)
@@
 			(at 194.31 113.03 90)
 			(hide yes)
+			(show_name no)
+			(do_not_autoplace no)
+			(effects
+				(font
+					(size 1.27 1.27)
+				)
+			)
+		)
+		(property "LCSC Part" "C23345"
+			(at 194.31 113.03 90)
+			(hide yes)
