File: pcb/clock.kicad_sch (KiCad schematic)
At the start: 5 parts, among them Y1 Crystal_GND24

Commit message: asigning the footprints
Parts:
- C4: renamed from C3; footprint Package_SON:Winbond_USON-8-1EP_3x2mm_P0.5mm_EP0.2x1.6mm -> Capacitor_SMD:C_0603_1608Metric; LCSC Part (none) -> C1644
- C5: renamed from C4; footprint Package_SON:Winbond_USON-8-1EP_3x2mm_P0.5mm_EP0.2x1.6mm -> Capacitor_SMD:C_0603_1608Metric; LCSC Part (none) -> C1644
- R10: renamed from R7; footprint (none) -> Resistor_SMD:R_0603_1608Metric
- R11: renamed from R6; value 1K -> 100; footprint Package_DIP:DIP-8_W7.62mm -> Resistor_SMD:R_0603_1608Metric
- Y1: value Crystal_GND24 -> 12Mhz; footprint (none) -> Crystal:Crystal_SMD_3225-4Pin_3.2x2.5mm

Commit message: asigning the part numbers
Parts:
- R10: LCSC Part (none) -> -
- R11: LCSC Part (none) -> C2906981
- Y1: LCSC Part (none) -> C2842186
Changed lines of the file:
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@@
+			)
+		)
+		(property "LCSC Part" "C2906981"
+			(at 154.94 74.93 0)
+			(hide yes)
+			(show_name no)
+			(do_not_autoplace no)
+			(effects
+				(font
+					(size 1.27 1.27)
+				)
 			)
 		)
@@
 			)
 		)
+		(property "LCSC Part" "C2842186"
+			(at 147.32 85.09 0)
+			(hide yes)
+			(show_name no)
+			(do_not_autoplace no)
+			(effects
+				(font
+					(size 1.27 1.27)
+				)
+			)
+		)
 		(pin "3"
 		)
@@
 			(at 147.32 69.85 90)
 			(hide yes)
+			(show_name no)
+			(do_not_autoplace no)
+			(effects
+				(font
+					(size 1.27 1.27)
+				)
+			)
+		)
+		(property "LCSC Part" "-"
+			(at 147.32 69.85 90)
+			(hide yes)

Commit message: fixing mistakes and adding some documents about the shematic
Parts:
- R11: value 100 -> 1k; LCSC Part C2906981 -> C22548
- Y1: LCSC Part C2842186 -> C20625731
Changed lines of the file:
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@@
 			)
 		)
-		(property "Value" "100"
+		(property "Value" "1k"
 			(at 157.48 76.1999 0)
 			(show_name no)
@@
 			)
 		)
-		(property "LCSC Part" "C2906981"
+		(property "LCSC Part" "C22548"
 			(at 154.94 74.93 0)
 			(hide yes)
@@
 			)
 		)
-		(property "LCSC Part" "C2842186"
-			(at 147.32 85.09 0)
-			(hide yes)
+		(property "LCSC Part" "C20625731"
+			(at 147.32 85.09 0)
+			(hide yes)
