File: pcb/usb.kicad_sch (KiCad schematic)
At the start: 9 parts, among them J1 USB_A, U4 AP2112K-3.3, U5 USBLC6-2SC6

Commit message: asigning the footprints
Parts:
- C6: footprint Package_SON:Winbond_USON-8-1EP_3x2mm_P0.5mm_EP0.2x1.6mm -> Capacitor_SMD:C_0603_1608Metric; LCSC Part (none) -> C19702
- C7: renamed from C5; footprint Package_SON:Winbond_USON-8-1EP_3x2mm_P0.5mm_EP0.2x1.6mm -> Capacitor_SMD:C_0603_1608Metric; LCSC Part (none) -> C1591
- C8: renamed from C7; footprint Package_SON:Winbond_USON-8-1EP_3x2mm_P0.5mm_EP0.2x1.6mm -> Capacitor_SMD:C_0603_1608Metric; LCSC Part (none) -> C19702
- C9: renamed from C8; footprint Package_SON:Winbond_USON-8-1EP_3x2mm_P0.5mm_EP0.2x1.6mm -> Capacitor_SMD:C_0603_1608Metric; LCSC Part (none) -> C1591
- J1: footprint (none) -> custom_lib:USB_A_PCB_Edge_receptacle
- R12: renamed from R9; footprint Package_TO_SOT_SMD:SOT-23-5 -> Resistor_SMD:R_0603_1608Metric
- R13: renamed from R8; footprint Package_TO_SOT_SMD:SOT-23-5 -> Resistor_SMD:R_0603_1608Metric
Connections:
- net GND: no longer J1.SH (Shield)
- net at J1.2 (D-), U5.4 (I/O2): no longer R13.1, U5.1 (I/O1)
- net at J1.3 (D+), U5.6 (I/O1): no longer R12.1, U5.3 (I/O2)
- new net: R13.1, U5.1 (I/O1)
- new net: R12.1, U5.3 (I/O2)
- no-connect marks 0 -> 1
Other:
- moved on the sheet: R12, R13

Commit message: asigning the part numbers
Parts:
- J1: LCSC Part (none) -> -
- R12, R13: LCSC Part (none) -> C2907021
- U4: LCSC Part (none) -> C51118
- U5: LCSC Part (none) -> C7519
Changed lines of the file:
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@@
+			)
+		)
+		(property "LCSC Part" "-"
+			(at 138.43 63.5 0)
+			(hide yes)
+			(show_name no)
+			(do_not_autoplace no)
+			(effects
+				(font
+					(size 1.27 1.27)
+				)
 			)
 		)
@@
 			)
 		)
+		(property "LCSC Part" "C7519"
+			(at 138.43 85.09 90)
+			(hide yes)
+			(show_name no)
+			(do_not_autoplace no)
+			(effects
+				(font
+					(size 1.27 1.27)
+				)
+			)
+		)
 		(pin "1"
 		)
@@
 			)
 		)
+		(property "LCSC Part" "C2907021"
+			(at 162.56 95.25 90)
+			(hide yes)
+			(show_name no)
+			(do_not_autoplace no)
+			(effects
+				(font
+					(size 1.27 1.27)
+				)
+			)
+		)
 		(pin "2"
 		)
@@
 		)
 		(property "KLC_S4.2_VREG_VOUT" ""
+			(at 162.56 90.17 90)
+			(hide yes)
+			(show_name no)
+			(do_not_autoplace no)
+			(effects
+				(font
+					(size 1.27 1.27)
+				)
+			)
+		)
+		(property "LCSC Part" "C2907021"
 			(at 162.56 90.17 90)
 			(hide yes)
@@
 			(at 130.81 123.19 90)
 			(hide yes)
+			(show_name no)
+			(do_not_autoplace no)
+			(effects
+				(font
+					(size 1.27 1.27)
+				)
+			)
+		)
+		(property "LCSC Part" "C51118"
+			(at 130.81 123.19 90)
+			(hide yes)

Commit message: Designing the usb data lanes
Parts:
- removed R12, R13: 27, Resistor_SMD:R_0603_1608Metric, symbol Device:R
- removed U5: USBLC6-2SC6, Package_TO_SOT_SMD:SOT-23-6, symbol Power_Protection:USBLC6-2SC6
- added D2: ESDS302DBVR, easyeda2kicad:SOT-23-5_L3.0-W1.6-P0.95-LS2.8-BL, symbol EasyKiCad:ESDS302DBVR
Connections:
- net D+: now also J1.2 (D-), D2.4 (I/O1)
- net D-: now also J1.3 (D+), D2.5 (I/O2)
- net GND: now also D2.2 (GND)
