File: pcb/pcb.kicad_pcb (KiCad board)
At the start: 4 copper layers, 60 x 14 mm, 37 parts, among them J1 USB_A, SW1 SW_Push, SW2 SW_Push, SW3 SW_Push_Big, U1 RP2040, U2 ATECC608A-SSHDA, U3 W25Q32JVSSIQ_C179173, U4 AP2112K-3.3, U5 USBLC6-2SC6, Y1 12Mhz

Commit message: doing the routing
Parts:
- removed R12, R13: 27, Resistor_SMD:R_0603_1608Metric
- removed U5: USBLC6-2SC6, Package_TO_SOT_SMD:SOT-23-6
- added C14: 100nF, Capacitor_SMD:C_0603_1608Metric, F.Cu at (87.7, 74.0)
- added C15: 100nF, Capacitor_SMD:C_0603_1608Metric, F.Cu at (98.2, 75.2)
- added C16: 100nF, Capacitor_SMD:C_0603_1608Metric, F.Cu at (96.0, 77.8)
- added D2: ESDS302DBVR, easyeda2kicad:SOT-23-5_L3.0-W1.6-P0.95-LS2.8-BL, F.Cu at (107.2, 74.0)
- moved R2 64.8 mm to (61.6, 71.0), turned to 90 degrees
- moved R1 63.5 mm to (75.0, 78.5)
- moved C13 58.2 mm to (91.6, 78.5), turned to 90 degrees
- moved C1 51.9 mm to (100.3, 71.8), turned to 90 degrees
- moved C8 49.6 mm to (102.9, 71.4), turned to 180 degrees
- moved R8 43.4 mm to (78.5, 73.9), turned to 90 degrees
- moved R9 41.9 mm to (80.3, 76.2), turned to 180 degrees
- moved U3 40.1 mm to (83.0, 79.5), turned to 90 degrees
- moved C9 34.3 mm to (102.9, 69.9), turned to 180 degrees
- moved C3 30.7 mm to (92.9, 67.3)
- moved C12 29.9 mm to (76.5, 81.5), turned to 180 degrees
- moved R5 24.8 mm to (68.4, 74.9)
- moved U2 24.2 mm to (76.1, 67.8)
- moved R6 21.7 mm to (68.4, 73.4)
- moved C2 20.8 mm to (81.3, 66.0)
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Connections:
- J1 pad 2: /usb/raw_D- -> /usb/D+
- J1 pad 3: /usb/raw_D+ -> /usb/D-
Routing:
- net /memory/CE: track 0.00 -> 45.0 mm
- net +3.3V: track 0.00 -> 40.0 mm, vias 0 -> 13
- net Net-(U1-GPIO7): track 0.00 -> 39.2 mm, vias 0 -> 2
- net /RGB/R: track 0.00 -> 30.8 mm, vias 0 -> 2
- net /usb/D+: track 0.00 -> 30.1 mm
- net /usb/D-: track 0.00 -> 30.1 mm
- net GND: track 16.8 -> 46.5 mm, vias 5 -> 44
- net /RGB/G: track 0.00 -> 27.6 mm, vias 0 -> 2
- net /memory/SIO1: track 0.00 -> 25.7 mm, vias 0 -> 2
- net /RGB/B: track 0.00 -> 24.8 mm, vias 0 -> 2
- net /memory/SIO0: track 0.00 -> 23.5 mm, vias 0 -> 2
- net /memory/SIO3: track 0.00 -> 21.2 mm, vias 0 -> 2
- net /Crypt/sda: track 0.00 -> 21.1 mm, vias 0 -> 3
- net /Crypt/scl: track 0.00 -> 19.3 mm, vias 0 -> 3
- net /usb/raw_D-: track 19.2 -> 0.00 mm
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Other:
- board size 60 x 14 mm -> 60.6 x 18 mm
