File: pcb/pcb.kicad_sch (KiCad schematic)
At the start: 7 parts, among them SW4 SW_Push, SW5 SW_Push, SW6 SW_Push, U1 RP2040

Commit message: asigning the footprints
Parts:
- C1: renamed from C9; footprint (none) -> Capacitor_SMD:C_0603_1608Metric; LCSC Part (none) -> C1592
- R1: renamed from R10; footprint (none) -> Resistor_SMD:R_0603_1608Metric
- R2: renamed from R11; footprint (none) -> Resistor_SMD:R_0603_1608Metric
- renumbered SW4 to SW1, SW5 to SW2, SW6 to SW3

Commit message: asigning the part numbers
Parts:
- R1: LCSC Part (none) -> C22548
- R2: LCSC Part (none) -> C98220
- SW3: value SW_Push -> SW_Push_Big; LCSC Part (none) -> C2689521
- U1: LCSC Part (none) -> C2040
Changed lines of the file:
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@@
+			)
+		)
+		(property "LCSC Part" "C22548"
+			(at 62.23 93.98 0)
+			(hide yes)
+			(show_name no)
+			(do_not_autoplace no)
+			(effects
+				(font
+					(size 1.27 1.27)
+				)
 			)
 		)
@@
 			)
 		)
+		(property "LCSC Part" "C98220"
+			(at 179.07 86.36 0)
+			(hide yes)
+			(show_name no)
+			(do_not_autoplace no)
+			(effects
+				(font
+					(size 1.27 1.27)
+				)
+			)
+		)
 		(pin "1"
 		)
@@
 			)
 		)
-		(property "Value" "SW_Push"
+		(property "Value" "SW_Push_Big"
 			(at 191.77 87.63 0)
 			(show_name no)
@@
 		)
 		(property "KLC_S4.2_VREG_VOUT" ""
+			(at 191.77 82.55 0)
+			(hide yes)
+			(show_name no)
+			(do_not_autoplace no)
+			(effects
+				(font
+					(size 1.27 1.27)
+				)
+			)
+		)
+		(property "LCSC Part" "C2689521"
 			(at 191.77 82.55 0)
 			(hide yes)
@@
 			(at 143.51 102.87 0)
 			(hide yes)
+			(show_name no)
+			(do_not_autoplace no)
+			(effects
+				(font
+					(size 1.27 1.27)
+				)
+			)
+		)
+		(property "LCSC Part" "C2040"
+			(at 143.51 102.87 0)
+			(hide yes)

Commit message: fixing mistakes and adding some documents about the shematic
Parts:
- added C13: 1uF, Capacitor_SMD:C_0603_1608Metric, symbol Device:C
- SW1, SW2: footprint Package_TO_SOT_SMD:SOT-23-6 -> easyeda2kicad:SW-SMD_L3.9-W3.0-P4.45; LCSC Part (none) -> C115357
- SW3: footprint Package_TO_SOT_SMD:SOT-23-6 -> easyeda2kicad:SW-SMD_L3.9-W3.0-P4.45; LCSC Part C2689521 -> C115357
Connections:
- net +3.3V: now also C13.2
- net GND: now also C1.2, C13.1

Commit message: doing the routing
Changed lines of the file:
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@@
-	(wire
-		(pts
-			(xy 146.05 30.48) (xy 146.05 57.15)
-		)
-		(stroke
-			(width 0)
-			(type default)
-		)
-	)
 	(wire
 		(pts
@@
 	(wire
 		(pts
+			(xy 135.89 30.48) (xy 146.05 30.48)
+		)
+		(stroke
+			(width 0)
+			(type default)
+		)
+	)
+	(wire
+		(pts
 			(xy 177.8 97.79) (xy 168.91 97.79)
 		)
@@
 	(wire
 		(pts
-			(xy 135.89 30.48) (xy 146.05 30.48)
+			(xy 179.07 82.55) (xy 168.91 82.55)
 		)
 		(stroke
@@
 	(wire
 		(pts
-			(xy 179.07 82.55) (xy 168.91 82.55)
+			(xy 146.05 30.48) (xy 146.05 57.15)
 		)
 		(stroke
@@
 		)
 	)
+	(label "Vreg_Vin"
+		(at 146.05 57.15 90)
+		(effects
+			(font
+				(size 1.27 1.27)
+			)
+			(justify left bottom)
+		)
+	)
